File: eagle/powerblade/powerblade_test.brd (EAGLE design)
At the start: 123 x 88 mm, 130 parts, among them J1 JTAG_14PIN_IDC-NL, J21 AC_INSW, Q1 2SK1829, Q2 2SK1829, U1 TPS62122, U2 TR1000, U3 MSP430FR5738, U4 LTC5800, U5 MAX9910, U6 MAX9910, U7 OPA2369, X1 ABM8G, X2 ABS07, Y1 UREACH_XTEND, Y2 ANT-916

Commit message: finished powerblade
Parts:
- added C34, C8: 8pF, rcl:C0603
- added LED2: (no value), SparkFun-LED:LED-0603
- added Q3: 2SK1829, powerfilm:SC-70-3
- added R11: 134k 1%, rcl:R0603
- added R12: 67k 1%, rcl:R0603
- added R23: 120, rcl:R0603
- added TP14: TP_STD, skyspecs:TP
- added X3: 32.768kHz, general:0805
- J1: value JTAG_14PIN_IDC-NL -> JTAG_14PIN_IDC; device ibat:TC2050-IDC-NL-430 -> ibat:TC2050-IDC-430
- R38: device rcl:R0402 -> rcl:R0603
- moved TP13 27.7 mm to (41.2, 75.4)
- moved TP12 23.0 mm to (41.2, 72.6)
- moved R34 19.8 mm to (31.0, 70.1), turned to 180 degrees
- moved TP10 14.1 mm to (20.8, 48.3)
- moved TP11 13.5 mm to (17.7, 48.3)
- moved R47 11.5 mm to (101.1, 79.1), turned to 90 degrees
- moved R43 8.00 mm to (105.3, 68.7), turned to 90 degrees
- moved J1 8.00 mm to (11.1, 73.7)
- moved R49 6.08 mm to (51.3, 54.6), turned to 90 degrees
- moved R33 6.01 mm to (27.5, 60.6), turned to 270 degrees
- moved R37 5.21 mm to (59.8, 64.3), turned to 180 degrees
- moved TP8 5.01 mm to (89.3, 64.8)
- moved C39 4.24 mm to (59.7, 66.0), turned to 270 degrees
- moved R45 4.17 mm to (104.2, 68.7), turned to 90 degrees
- moved C38 3.72 mm to (62.2, 61.4), turned to 270 degrees
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Connections:
- net N$2 renamed N
- net N$6 renamed P
- removed net LED_EN: Q2.P1, U3.P16
- new net N$1: C34.2, U3.P22, X3.1
- new net N$56: C8.2, U3.P21, X3.2
- new net N$58: LED2.A, R23.1
- new net N$59: LED2.C, Q3.P3
- new net VCC_SENSE: R11.1, R12.2, U3.P4
- net +3V3: now also R23.2
- net GND: now also C34.1, C8.1, Q3.P2, R12.1, TP14.P$1
- net I_SENSE: now also U4.P18; no longer U4.P17
- net RXDATA: now also U3.P16; no longer U3.P4
- net TCK: now also Q2.P1
- net TDI: now also Q3.P1
- net VCC: now also R11.2
- net V_SENSE: now also U4.P17; no longer U4.P15
Routing:
- net +3V3: track 0.00 -> 349.8 mm, vias 0 -> 16
- net I_SENSE: track 0.00 -> 148.8 mm
- net V_SENSE: track 0.00 -> 135.9 mm, vias 0 -> 2
- net LTC_RX: track 0.00 -> 119.6 mm, vias 0 -> 4
- net LTC_TX: track 0.00 -> 107.9 mm
- net LTC_SLEEP: track 0.00 -> 107.5 mm, vias 0 -> 2
- net P: track 0.00 -> 102.1 mm, vias 1 -> 3
- net N: track 0.00 -> 87.0 mm, vias 1 -> 2
- net DGND: track 0.00 -> 81.3 mm, vias 0 -> 10
- net VCC_SENSE: track 0.00 -> 68.3 mm, vias 0 -> 2
- net VTEST: track 0.00 -> 50.1 mm, vias 0 -> 1
- net METER_EN: track 0.00 -> 48.7 mm, vias 0 -> 2
- net TCK: track 0.00 -> 47.6 mm, vias 0 -> 2
- net RXDATA: track 0.00 -> 46.1 mm, vias 0 -> 1
- net N$67: track 0.00 -> 45.6 mm, vias 0 -> 3
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- added copper zone on layer 16, net +3V3
- added copper zone on layer 16, net DGND
- added copper zone on layer 16, net N$34
- added copper zone on layer 16, net N$35
- added copper zone on layer 16, net N$4
- added copper zone on layer 16, net N$41
Other:
- board text added: "+3v3"
- board text added: "2/27/15"
- board text added: "2v0"
- board text added: "AMP"
- board text added: "CS+"
- board text added: "FILT"
- board text added: "GND"
- board text added: "HV"
- board text added: "IS"
- board text added: "N"
- board text added: "P"
- board text added: "PowerBlade Test"
- board text added: "Sam DeBruin"
- board text added: "VCC"
- board text added: "VS"

Commit message: finished doing parts for powerblade test
Parts:
- R31, R32: value 4.99k -> 47k
- R46, R48: value 33k -> 47k
- R47: value 33k -> 12k
