File: eagle/powerblade/powerblade_3v2.sch (EAGLE design)
At the start: 78 parts, among them J1 JTAG_14PIN_IDC-ND, J2 AC_INF4, J4 TC2030-JLINK-NL, Q1 NTS4173, Q4 2SK1829, U1 TPS62122, U2 MCP6V3, U3 MSP430FR5738, U4 NRF51822QF, U6 MAX9910, U7 OPA2369, X1 16MHz, X3 32.768kHz, Y1 UREACH_XTEND

Commit message: updated l41
Parts:
- J2: value AC_INF4 -> AC_INF41; device powerfilm:AC_INF4 -> powerfilm:AC_INF41
Changed lines of the file:
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@@
 <?xml version="1.0" encoding="utf-8"?>
 <!DOCTYPE eagle SYSTEM "eagle.dtd">
-<eagle version="6.5.0">
+<eagle version="6.3">
 <drawing>
 <settings>
@@
 <attribute name="DIGIKEY" value="490-4025-1-ND"/>
 </part>
-<part name="J2" library="powerfilm" deviceset="AC_IN" device="F4" value="AC_INF4">
+<part name="J2" library="powerfilm" deviceset="AC_IN" device="F41" value="AC_INF41">
 <attribute name="DIGIKEY" value="ED1649-ND"/>
 <attribute name="DIGIKEY_2" value="ED1649-ND"/>

Commit message: updated board? I hope i dont get conflicts
Parts:
- J2: value AC_INF41 -> AC_INF45; device powerfilm:AC_INF41 -> powerfilm:AC_INF45
Changed lines of the file:
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@@
 <attribute name="DIGIKEY" value="490-4025-1-ND"/>
 </part>
-<part name="J2" library="powerfilm" deviceset="AC_IN" device="F41" value="AC_INF41">
+<part name="J2" library="powerfilm" deviceset="AC_IN" device="F45" value="AC_INF45">
 <attribute name="DIGIKEY" value="ED1649-ND"/>
 <attribute name="DIGIKEY_2" value="ED1649-ND"/>
