File: eagle/inductor_test/inductor_test_2v0.brd (EAGLE design)
At the start: 25.4 x 50.8 mm, 82 parts, among them J1 MA02-1, U1 OPA2369, U2 OPA2369, U3 SC70, U4 SOT-23-6, U5 TSSOP-14, U6 TPS62122, U7 MAX9910

Commit message: added part numbers and values
Parts:
- C1, C6, C7, C8: value (none) -> 1.5uF
- C10, C11, C12, C13, C2, C9: value (none) -> Sh/10uF
- C14, C15, C3, C4, C5: value (none) -> 0.1uF
- R1, R12, R13, R5: value (none) -> 20k
- R10, R6, R9: value (none) -> 4.99k/1.3M
- R11, R7, R8: value (none) -> 4.99/1k
- R14, R16, R18: value (none) -> 887k
- R15, R17, R19: value (none) -> 30k/29.8k
- R20, R21, R22: value (none) -> 100k
- R23: value (none) -> 1.6k
- R31: value (none) -> 240

Commit message: finished adding part numbers for inductor test board
Parts:
- R20, R21, R22: value 100k -> 1M
- R23: value 1.6k -> 16k
